File: all in one/all-in-one.brd (EAGLE design)
At the start: 100 x 80 mm, 89 parts, among them J1 K1, J10 DIN, J11 START, J12 SELECT, J13 HOME, J14 BALLTOP, J15 PLATE, J2 P1, J20 DOUT, J21 led, J3 K2, J4 P2, J5 K3, J6 P3, J7 K4, J8 P4, J9 led

Commit message: rooby dooby dooby
Parts:
- moved C15 14.9 mm to (76.0, 53.0)
- moved C16 14.9 mm to (82.0, 53.0)
- moved J8 14.9 mm to (80.0, 63.0)
- moved L15 14.9 mm to (76.0, 58.0)
- moved L16 14.9 mm to (82.0, 58.0)
- moved C11 14.2 mm to (63.0, 53.0)
- moved C12 14.2 mm to (69.0, 53.0)
- moved J6 14.2 mm to (67.0, 63.0)
- moved L11 14.2 mm to (63.0, 58.0)
- moved L12 14.2 mm to (69.0, 58.0)
- moved C7 13.6 mm to (50.0, 53.0)
- moved C8 13.6 mm to (56.0, 53.0)
- moved J10 13.6 mm to (79.0, 28.0)
- moved J4 13.6 mm to (54.0, 63.0)
- moved J9 13.6 mm to (84.0, 28.0)
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Routing:
- net VCC: track 524.4 -> 471.3 mm
- net UP: track 61.5 -> 54.5 mm
- net RIGHT: track 51.6 -> 44.6 mm
- net LEFT: track 60.5 -> 53.5 mm
- net DOWN: track 61.0 -> 54.0 mm
Other:
- board size 100 x 80 mm -> 87 x 67 mm
- board text added: "+"
- board text added: "-"
- board text added: "1P ST"
- board text added: "2K 1K"
- board text added: "3P 2P"
- board text added: "4K 3K"
- board text added: "4P -"
- board text added: "BALL"
- board text added: "DN UP"
- board text added: "HO SE"
- board text added: "HOME"
- board text added: "K1"
- board text added: "K2"
- board text added: "K3"
- board text added: "K4"
- board text added: "LT RT"
- board text added: "P1"
- board text added: "P2"
- board text added: "P3"
- board text added: "P4"
- board text added: "PLATE"
- board text added: "SEL"
- board text added: "STA"

Commit message: Tue Mar  7 09:28:05 EST 2017
Parts:
- added LED1: (no value), led:CHIPLED_0805
- added R1: (no value), adafruit:R0805
- S1, S10, S11, S12, S13, S14, S15, S2, S3, S4, S5, S6, S7, S8, S9: device SparkFun-Electromechanical:TACTILE-SWITCH-SMD -> SparkFun-Switches:TACTILE_SWITCH_SMD_4.5MM
- turned S1 to 90 degrees
- turned S10 to 270 degrees
- turned S11 to 270 degrees
- turned S12 to 270 degrees
- turned S13 to 270 degrees
- turned S14 to 270 degrees
- turned S15 to 270 degrees
- turned S2 to 90 degrees
- turned S3 to 90 degrees
- turned S4 to 90 degrees
- turned S5 to 270 degrees
- turned S6 to 270 degrees
- turned S7 to 270 degrees
- turned S8 to 270 degrees
- turned S9 to 270 degrees
Connections:
- new net N$37: LED1.A, R1.2
- net 1K: now also S5.1, S5.4; no longer S5.3
- net 1P: now also S1.1, S1.4; no longer S1.3
- net 2K: now also S6.1, S6.4; no longer S6.3
- net 2P: now also S2.1, S2.4; no longer S2.3
- net 3K: now also S7.1, S7.4; no longer S7.3
- net 3P: now also S3.1, S3.4; no longer S3.3
- net 4K: now also S8.1, S8.4; no longer S8.3
- net 4P: now also S4.1, S4.4; no longer S4.3
- net DOWN: now also S13.1, S13.4; no longer S13.3
- net GND: now also LED1.C, S1.2, S1.3, S10.2, S10.3, S11.2, S11.3, S12.2, S12.3, S13.2, S13.3, S14.2, S14.3, S15.2, S15.3, S2.2, S2.3, S3.2, S3.3, S4.2, S4.3, S5.2, S5.3, S6.2, S6.3, S7.2, S7.3, S8.2, S8.3, S9.2, S9.3; no longer S1.1, S10.1, S11.1, S12.1, S13.1, S14.1, S15.1, S2.1, S3.1, S4.1, S5.1, S6.1, S7.1, S8.1, S9.1
- net HOME: now also S11.1, S11.4; no longer S11.3
- net LEFT: now also S14.1, S14.4; no longer S14.3
- net RIGHT: now also S15.1, S15.4; no longer S15.3
- net SELECT: now also S10.1, S10.4; no longer S10.3
- net START: now also S9.1, S9.4; no longer S9.3
- net UP: now also S12.1, S12.4; no longer S12.3
- net VCC: now also R1.1
Routing:
- net SELECT: track 11.0 -> 37.7 mm, vias 0 -> 2
- net HOME: track 11.4 -> 32.2 mm, vias 0 -> 2
- net START: track 19.9 -> 33.7 mm, vias 0 -> 2
- net RIGHT: track 44.6 -> 58.2 mm, vias 0 -> 2
- net 4P: track 65.3 -> 70.5 mm, vias 2 -> 1
- net UP: track 54.5 -> 59.7 mm
- net 3P: track 52.8 -> 57.9 mm
- net 2P: track 45.9 -> 50.8 mm
- net 4K: track 54.7 -> 59.6 mm
- net 3K: track 51.3 -> 56.1 mm
- net 1K: track 37.7 -> 42.6 mm
- net 2K: track 40.7 -> 45.5 mm
- net VCC: track 471.3 -> 468.0 mm
- net N$37: track 0.00 -> 2.05 mm
- net 1P: track 32.8 -> 34.6 mm
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Other:
- board text added: "CONNECT FROM BOTTOM ONLY!"
