File: Gameboy Pocket/Gameboy Pocket.sch (EAGLE design)
At the start: 34 parts, among them CN1 USB-SMD-NS, J3 battery, X3 16MHz

Commit message: Fri Mar 10 05:58:47 EST 2017
Parts:
- added J1: (no value), SparkFun-Connectors:CONN_08NO_SILK_FEMALE_PTH
Connections:
- new net HWB: U$2.PE2/!HWB
- net A0: now also J1.8
- net A1: now also J1.7
- net A2: now also J1.6
- net A3: now also J1.5
- net A4: now also J1.4
- net A5: now also J1.3
- net D11: now also J1.2
- net D7: now also J1.1
