File: Gameboy Pocket/Gameboy Pocket.sch (EAGLE design)
At the start: 35 parts, among them CN1 USB-SMD-NS, J3 battery, X3 16MHz

Commit message: Wed Mar 15 19:26:25 EDT 2017
Parts:
- J1: device SparkFun-Connectors:CONN_08NO_SILK_FEMALE_PTH -> SparkFun-Connectors:CONN_07NO_SILK
- J3: device SparkFun-Connectors:M02JST-PTH-VERT -> SparkFun-Connectors:M021X02_NO_SILK
- JP2: value (none) -> Speaker; device SparkFun-Connectors:M02PTH -> SparkFun-Connectors:M021X02_NO_SILK
Connections:
- removed net A0: J1.8, U$2.PF7(ADC7)
- removed net SPEAKER: JP2.2
- new net A0/SPEAKER: JP2.2, U$2.PF7(ADC7)
